File: pcb/sunboard/LED_Matrix.kicad_sch (KiCad schematic)
At the start: 0 parts

Commit message: feat(pcb): remove led driver, layout main grid
Parts:
- added D1, D10, D100, D101, D102, D103, D104, D105, D106, D107, D108, D109, D11, D110, D111, D112, D113, D114, D115, D116, D117, D118, D119, D12, D120, D121, D122, D123, D124, D125, D126, D127, D128, D129, D13, D130, D131, D132, D133, D134, D135, D136, D137, D138, D139, D14, D140, D141, D142, D143, D144, D145, D146, D147, D148, D149, D15, D150, D151, D152, D153, D154, D16, D17, D18, D19, D2, D20, D21, D22, D23, D24, D25, D26, D27, D28, D29, D3, D30, D31, D32, D33, D34, D35, D36, D37, D38, D39, D4, D40, D41, D42, D43, D44, D45, D46, D47, D48, D49, D5, D50, D51, D52, D53, D54, D55, D56, D57, D58, D59, D6, D60, D61, D62, D63, D64, D65, D66, D67, D68, D69, D7, D70, D71, D72, D73, D74, D75, D76, D77, D78, D79, D8, D80, D81, D82, D83, D84, D85, D86, D87, D88, D89, D9, D90, D91, D92, D93, D94, D95, D96, D97, D98, D99: WS2812B, LED_SMD:LED_WS2812B_PLCC4_5.0x5.0mm_P3.2mm, symbol LED:WS2812B
Connections:
- new net: D49.2 (DOUT), D50.4 (DIN)
- new net: D48.2 (DOUT), D49.4 (DIN)
- new net: D31.2 (DOUT), D32.4 (DIN)
- new net: D30.2 (DOUT), D31.4 (DIN)
- new net: D90.2 (DOUT), D91.4 (DIN)
- new net: D89.2 (DOUT), D90.4 (DIN)
- new net: D41.2 (DOUT), D42.4 (DIN)
- new net: D40.2 (DOUT), D41.4 (DIN)
- new net: D29.2 (DOUT), D30.4 (DIN)
- new net: D81.2 (DOUT), D82.4 (DIN)
- new net: D80.2 (DOUT), D81.4 (DIN)
- new net: D84.2 (DOUT), D85.4 (DIN)
- new net: D83.2 (DOUT), D84.4 (DIN)
- new net: D128.2 (DOUT), D129.4 (DIN)
- new net: D127.2 (DOUT), D128.4 (DIN)
- new net: D33.2 (DOUT), D34.4 (DIN)
- new net: D32.2 (DOUT), D33.4 (DIN)
- new net: D3.2 (DOUT), D4.4 (DIN)
- new net: D2.2 (DOUT), D3.4 (DIN)
- new net: D43.2 (DOUT), D44.4 (DIN)
- new net: D42.2 (DOUT), D43.4 (DIN)
- new net: D85.2 (DOUT), D86.4 (DIN)
- new net: D25.2 (DOUT), D26.4 (DIN)
- new net: D24.2 (DOUT), D25.4 (DIN)
- new net: D76.2 (DOUT), D77.4 (DIN)
- new net: D75.2 (DOUT), D76.4 (DIN)
- new net: D153.2 (DOUT), D154.4 (DIN)
- new net: D152.2 (DOUT), D153.4 (DIN)
- new net: D140.2 (DOUT), D141.4 (DIN)
- new net: D139.2 (DOUT), D140.4 (DIN)
- new net: D136.2 (DOUT), D137.4 (DIN)
- new net: D135.2 (DOUT), D136.4 (DIN)
- new net: D8.2 (DOUT), D9.4 (DIN)
- new net: D7.2 (DOUT), D8.4 (DIN)
- new net: D98.2 (DOUT), D99.4 (DIN)
- new net: D97.2 (DOUT), D98.4 (DIN)
- new net: D53.2 (DOUT), D54.4 (DIN)
- new net: D52.2 (DOUT), D53.4 (DIN)
- new net: D145.2 (DOUT), D146.4 (DIN)
- new net: D144.2 (DOUT), D145.4 (DIN)
- new net: D71.2 (DOUT), D72.4 (DIN)
- new net: D70.2 (DOUT), D71.4 (DIN)
- new net: D17.2 (DOUT), D18.4 (DIN)
- new net: D16.2 (DOUT), D17.4 (DIN)
- new net: D77.2 (DOUT), D78.4 (DIN)
- new net: D110.2 (DOUT), D111.4 (DIN)
- new net: D109.2 (DOUT), D110.4 (DIN)
- new net: D12.2 (DOUT), D13.4 (DIN)
- new net: D11.2 (DOUT), D12.4 (DIN)
- new net: D96.2 (DOUT), D97.4 (DIN)
- new net: D119.2 (DOUT), D120.4 (DIN)
- new net: D118.2 (DOUT), D119.4 (DIN)
- new net: D88.2 (DOUT), D89.4 (DIN)
- new net: D87.2 (DOUT), D88.4 (DIN)
- new net: D114.2 (DOUT), D115.4 (DIN)
- new net: D113.2 (DOUT), D114.4 (DIN)
- new net: D115.2 (DOUT), D116.4 (DIN)
- new net: D79.2 (DOUT), D80.4 (DIN)
- new net: D69.2 (DOUT), D70.4 (DIN)
- new net: D104.2 (DOUT), D105.4 (DIN)
- new net: D103.2 (DOUT), D104.4 (DIN)
- new net: D62.2 (DOUT), D63.4 (DIN)
- new net: D61.2 (DOUT), D62.4 (DIN)
- new net: D23.2 (DOUT), D24.4 (DIN)
- new net: D1.2 (DOUT), D2.4 (DIN)
- new net: D101.2 (DOUT), D102.4 (DIN)
- new net: D100.2 (DOUT), D101.4 (DIN)
- new net: D102.2 (DOUT), D103.4 (DIN)
- new net: D149.2 (DOUT), D150.4 (DIN)
- new net: D148.2 (DOUT), D149.4 (DIN)
- new net: D68.2 (DOUT), D69.4 (DIN)
- new net: D67.2 (DOUT), D68.4 (DIN)
- new net: D54.2 (DOUT), D55.4 (DIN)
- new net: D14.2 (DOUT), D15.4 (DIN)
- new net: D13.2 (DOUT), D14.4 (DIN)
- new net: D100.4 (DIN), D99.2 (DOUT)
- new net: D142.2 (DOUT), D143.4 (DIN)
- new net: D141.2 (DOUT), D142.4 (DIN)
- new net: D123.2 (DOUT), D124.4 (DIN)
- new net: D122.2 (DOUT), D123.4 (DIN)
- new net: D151.2 (DOUT), D152.4 (DIN)
- new net: D59.2 (DOUT), D60.4 (DIN)
- new net: D58.2 (DOUT), D59.4 (DIN)
- new net: D47.2 (DOUT), D48.4 (DIN)
- new net: D78.2 (DOUT), D79.4 (DIN)
- new net: D147.2 (DOUT), D148.4 (DIN)
- new net: D146.2 (DOUT), D147.4 (DIN)
- new net: D130.2 (DOUT), D131.4 (DIN)
- new net: D129.2 (DOUT), D130.4 (DIN)
- new net: D46.2 (DOUT), D47.4 (DIN)
- new net: D45.2 (DOUT), D46.4 (DIN)
- new net: D150.2 (DOUT), D151.4 (DIN)
- new net: D65.2 (DOUT), D66.4 (DIN)
- new net: D64.2 (DOUT), D65.4 (DIN)
- new net: D143.2 (DOUT), D144.4 (DIN)
- new net: D95.2 (DOUT), D96.4 (DIN)
- new net: D94.2 (DOUT), D95.4 (DIN)
- new net: D126.2 (DOUT), D127.4 (DIN)
- new net: D19.2 (DOUT), D20.4 (DIN)
- new net: D18.2 (DOUT), D19.4 (DIN)
- new net: D108.2 (DOUT), D109.4 (DIN)
- new net: D107.2 (DOUT), D108.4 (DIN)
- new net: D10.2 (DOUT), D11.4 (DIN)
- new net: D20.2 (DOUT), D21.4 (DIN)
- new net: D93.2 (DOUT), D94.4 (DIN)
- new net: D92.2 (DOUT), D93.4 (DIN)
- new net: D132.2 (DOUT), D133.4 (DIN)
- new net: D131.2 (DOUT), D132.4 (DIN)
- new net: D137.2 (DOUT), D138.4 (DIN)
- new net: D44.2 (DOUT), D45.4 (DIN)
- new net: D91.2 (DOUT), D92.4 (DIN)
- new net: D10.4 (DIN), D9.2 (DOUT)
- new net: D112.2 (DOUT), D113.4 (DIN)
- new net: D111.2 (DOUT), D112.4 (DIN)
- new net: D56.2 (DOUT), D57.4 (DIN)
- new net: D55.2 (DOUT), D56.4 (DIN)
- new net: D86.2 (DOUT), D87.4 (DIN)
- new net: D74.2 (DOUT), D75.4 (DIN)
- new net: D73.2 (DOUT), D74.4 (DIN)
- new net: D138.2 (DOUT), D139.4 (DIN)
- new net: D72.2 (DOUT), D73.4 (DIN)
- new net: D6.2 (DOUT), D7.4 (DIN)
- new net: D5.2 (DOUT), D6.4 (DIN)
- new net: D125.2 (DOUT), D126.4 (DIN)
- new net: D124.2 (DOUT), D125.4 (DIN)
- new net: D106.2 (DOUT), D107.4 (DIN)
- new net: D4.2 (DOUT), D5.4 (DIN)
- new net: D21.2 (DOUT), D22.4 (DIN)
- new net: D51.2 (DOUT), D52.4 (DIN)
- new net: D117.2 (DOUT), D118.4 (DIN)
- new net: D116.2 (DOUT), D117.4 (DIN)
- new net: D82.2 (DOUT), D83.4 (DIN)
- new net: D57.2 (DOUT), D58.4 (DIN)
- new net: D134.2 (DOUT), D135.4 (DIN)
- new net: D105.2 (DOUT), D106.4 (DIN)
- new net: D63.2 (DOUT), D64.4 (DIN)
- new net: D121.2 (DOUT), D122.4 (DIN)
- new net: D66.2 (DOUT), D67.4 (DIN)
- new net: D133.2 (DOUT), D134.4 (DIN)
- new net: D34.2 (DOUT), D35.4 (DIN)
- new net: D60.2 (DOUT), D61.4 (DIN)
- new net: D15.2 (DOUT), D16.4 (DIN)
- new net: D39.2 (DOUT), D40.4 (DIN)
- new net: D38.2 (DOUT), D39.4 (DIN)
- new net: D22.2 (DOUT), D23.4 (DIN)
- new net: D27.2 (DOUT), D28.4 (DIN)
- new net: D26.2 (DOUT), D27.4 (DIN)
- new net: D50.2 (DOUT), D51.4 (DIN)
- new net: D35.2 (DOUT), D36.4 (DIN)
- new net: D36.2 (DOUT), D37.4 (DIN)
- new net: D120.2 (DOUT), D121.4 (DIN)
- new net: D37.2 (DOUT), D38.4 (DIN)
- new net: D28.2 (DOUT), D29.4 (DIN)
- new net +5V: D1.1 (VDD), D10.1 (VDD), D100.1 (VDD), D101.1 (VDD), D102.1 (VDD), D103.1 (VDD), D104.1 (VDD), D105.1 (VDD), D106.1 (VDD), D107.1 (VDD), D108.1 (VDD), D109.1 (VDD), D11.1 (VDD), D110.1 (VDD), D111.1 (VDD), D112.1 (VDD), D113.1 (VDD), D114.1 (VDD), D115.1 (VDD), D116.1 (VDD), D117.1 (VDD), D118.1 (VDD), D119.1 (VDD), D12.1 (VDD), D120.1 (VDD), D121.1 (VDD), D122.1 (VDD), D123.1 (VDD), D124.1 (VDD), D125.1 (VDD), D126.1 (VDD), D127.1 (VDD), D128.1 (VDD), D129.1 (VDD), D13.1 (VDD), D130.1 (VDD), D131.1 (VDD), D132.1 (VDD), D133.1 (VDD), D134.1 (VDD), D135.1 (VDD), D136.1 (VDD), D137.1 (VDD), D138.1 (VDD), D139.1 (VDD), D14.1 (VDD), D140.1 (VDD), D141.1 (VDD), D142.1 (VDD), D143.1 (VDD), D144.1 (VDD), D145.1 (VDD), D146.1 (VDD), D147.1 (VDD), D148.1 (VDD), D149.1 (VDD), D15.1 (VDD), D150.1 (VDD), D151.1 (VDD), D152.1 (VDD), D153.1 (VDD), D154.1 (VDD), D16.1 (VDD), D17.1 (VDD), D18.1 (VDD), D19.1 (VDD), D2.1 (VDD), D20.1 (VDD), D21.1 (VDD), D22.1 (VDD), D23.1 (VDD), D24.1 (VDD), D25.1 (VDD), D26.1 (VDD), D27.1 (VDD), D28.1 (VDD), D29.1 (VDD), D3.1 (VDD), D30.1 (VDD), D31.1 (VDD), D32.1 (VDD), D33.1 (VDD), D34.1 (VDD), D35.1 (VDD), D36.1 (VDD), D37.1 (VDD), D38.1 (VDD), D39.1 (VDD), D4.1 (VDD), D40.1 (VDD), D41.1 (VDD), D42.1 (VDD), D43.1 (VDD), D44.1 (VDD), D45.1 (VDD), D46.1 (VDD), D47.1 (VDD), D48.1 (VDD), D49.1 (VDD), D5.1 (VDD), D50.1 (VDD), D51.1 (VDD), D52.1 (VDD), D53.1 (VDD), D54.1 (VDD), D55.1 (VDD), D56.1 (VDD), D57.1 (VDD), D58.1 (VDD), D59.1 (VDD), D6.1 (VDD), D60.1 (VDD), D61.1 (VDD), D62.1 (VDD), D63.1 (VDD), D64.1 (VDD), D65.1 (VDD), D66.1 (VDD), D67.1 (VDD), D68.1 (VDD), D69.1 (VDD), D7.1 (VDD), D70.1 (VDD), D71.1 (VDD), D72.1 (VDD), D73.1 (VDD), D74.1 (VDD), D75.1 (VDD), D76.1 (VDD), D77.1 (VDD), D78.1 (VDD), D79.1 (VDD), D8.1 (VDD), D80.1 (VDD), D81.1 (VDD), D82.1 (VDD), D83.1 (VDD), D84.1 (VDD), D85.1 (VDD), D86.1 (VDD), D87.1 (VDD), D88.1 (VDD), D89.1 (VDD), D9.1 (VDD), D90.1 (VDD), D91.1 (VDD), D92.1 (VDD), D93.1 (VDD), D94.1 (VDD), D95.1 (VDD), D96.1 (VDD), D97.1 (VDD), D98.1 (VDD), D99.1 (VDD)
- new net GND: D1.3 (VSS), D10.3 (VSS), D100.3 (VSS), D101.3 (VSS), D102.3 (VSS), D103.3 (VSS), D104.3 (VSS), D105.3 (VSS), D106.3 (VSS), D107.3 (VSS), D108.3 (VSS), D109.3 (VSS), D11.3 (VSS), D110.3 (VSS), D111.3 (VSS), D112.3 (VSS), D113.3 (VSS), D114.3 (VSS), D115.3 (VSS), D116.3 (VSS), D117.3 (VSS), D118.3 (VSS), D119.3 (VSS), D12.3 (VSS), D120.3 (VSS), D121.3 (VSS), D122.3 (VSS), D123.3 (VSS), D124.3 (VSS), D125.3 (VSS), D126.3 (VSS), D127.3 (VSS), D128.3 (VSS), D129.3 (VSS), D13.3 (VSS), D130.3 (VSS), D131.3 (VSS), D132.3 (VSS), D133.3 (VSS), D134.3 (VSS), D135.3 (VSS), D136.3 (VSS), D137.3 (VSS), D138.3 (VSS), D139.3 (VSS), D14.3 (VSS), D140.3 (VSS), D141.3 (VSS), D142.3 (VSS), D143.3 (VSS), D144.3 (VSS), D145.3 (VSS), D146.3 (VSS), D147.3 (VSS), D148.3 (VSS), D149.3 (VSS), D15.3 (VSS), D150.3 (VSS), D151.3 (VSS), D152.3 (VSS), D153.3 (VSS), D154.3 (VSS), D16.3 (VSS), D17.3 (VSS), D18.3 (VSS), D19.3 (VSS), D2.3 (VSS), D20.3 (VSS), D21.3 (VSS), D22.3 (VSS), D23.3 (VSS), D24.3 (VSS), D25.3 (VSS), D26.3 (VSS), D27.3 (VSS), D28.3 (VSS), D29.3 (VSS), D3.3 (VSS), D30.3 (VSS), D31.3 (VSS), D32.3 (VSS), D33.3 (VSS), D34.3 (VSS), D35.3 (VSS), D36.3 (VSS), D37.3 (VSS), D38.3 (VSS), D39.3 (VSS), D4.3 (VSS), D40.3 (VSS), D41.3 (VSS), D42.3 (VSS), D43.3 (VSS), D44.3 (VSS), D45.3 (VSS), D46.3 (VSS), D47.3 (VSS), D48.3 (VSS), D49.3 (VSS), D5.3 (VSS), D50.3 (VSS), D51.3 (VSS), D52.3 (VSS), D53.3 (VSS), D54.3 (VSS), D55.3 (VSS), D56.3 (VSS), D57.3 (VSS), D58.3 (VSS), D59.3 (VSS), D6.3 (VSS), D60.3 (VSS), D61.3 (VSS), D62.3 (VSS), D63.3 (VSS), D64.3 (VSS), D65.3 (VSS), D66.3 (VSS), D67.3 (VSS), D68.3 (VSS), D69.3 (VSS), D7.3 (VSS), D70.3 (VSS), D71.3 (VSS), D72.3 (VSS), D73.3 (VSS), D74.3 (VSS), D75.3 (VSS), D76.3 (VSS), D77.3 (VSS), D78.3 (VSS), D79.3 (VSS), D8.3 (VSS), D80.3 (VSS), D81.3 (VSS), D82.3 (VSS), D83.3 (VSS), D84.3 (VSS), D85.3 (VSS), D86.3 (VSS), D87.3 (VSS), D88.3 (VSS), D89.3 (VSS), D9.3 (VSS), D90.3 (VSS), D91.3 (VSS), D92.3 (VSS), D93.3 (VSS), D94.3 (VSS), D95.3 (VSS), D96.3 (VSS), D97.3 (VSS), D98.3 (VSS), D99.3 (VSS)
- new net LED_IN: D1.4 (DIN)
- no-connect marks 0 -> 1

Commit message: feat(pcb): add display
Parts:
- D1, D10, D100, D101, D102, D103, D104, D105, D106, D107, D108, D109, D11, D110, D111, D112, D113, D114, D115, D116, D117, D118, D119, D12, D120, D121, D122, D123, D124, D125, D126, D127, D128, D129, D13, D130, D131, D132, D133, D134, D135, D136, D137, D138, D139, D14, D140, D141, D142, D143, D144, D145, D146, D147, D148, D149, D15, D150, D151, D152, D153, D154, D16, D17, D18, D19, D2, D20, D21, D22, D23, D24, D25, D26, D27, D28, D29, D3, D30, D31, D32, D33, D34, D35, D36, D37, D38, D39, D4, D40, D41, D42, D43, D44, D45, D46, D47, D48, D49, D5, D50, D51, D52, D53, D54, D55, D56, D57, D58, D59, D6, D60, D61, D62, D63, D64, D65, D66, D67, D68, D69, D7, D70, D71, D72, D73, D74, D75, D76, D77, D78, D79, D8, D80, D81, D82, D83, D84, D85, D86, D87, D88, D89, D9, D90, D91, D92, D93, D94, D95, D96, D97, D98, D99: JLCPCB Part # (none) -> C2843785
